File: FootForceSensor_ver1_0.sch (EAGLE design)
At the start: 69 parts, among them IC1 HX711, IC2 HX711, IC3 HX711, IC4 HX711, IC5 ADM3078E, M1 PRO_MICRO_THROUGH_HOLE, T1 MMBT3906, T2 MMBT3906, T3 MMBT3906, T4 MMBT3906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

Commit message: Maintenance of README and other public information
Other:
- note added: "1.0"
- note added: "1/1"
- note added: "August 7, 2022"
- note added: "FootForceSensor"
- moved on the sheet: C1, C10, C11, C12, C13, C14, C15, C16, C17, C18, C19, C2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
